Commit message: 06 - Simulate Your Robot with Gazebo

File: src/my_robot_description/urdf/common_properties.xacro (robot description, xacro)
@@ -7,3 +7,30 @@
         <color rgba="0.5 0.5 0.5 1" />
     </material>
+    <xacro:macro name="box_inertia" params="m l w h xyz rpy">
+        <inertial>
+            <origin xyz="${xyz}" rpy="${rpy}" />
+            <mass value="${m}" />
+            <inertia ixx="${(m/12)*(h*h + l*l)}" ixy="0" ixz="0"
+                iyy="${(m/12)*(w*w + l*l)}" iyz="0"
+                izz="${(m/12)*(w*w + h*h)}" />
+        </inertial>
+    </xacro:macro>
+    <xacro:macro name="cylinder_inertia" params="m r h xyz rpy">
+        <inertial>
+            <origin xyz="${xyz}" rpy="${rpy}" />
+            <mass value="${m}" />
+            <inertia ixx="${(m/12)*(3*r*r + h*h)}" ixy="0" ixz="0"
+                iyy="${(m/12)*(3*r*r + h*h)}" iyz="0"
+                izz="${(m*r*r)/2}" />
+        </inertial>
+    </xacro:macro>
+    <xacro:macro name="sphere_inertia" params="m r xyz rpy">
+        <inertial>
+            <origin xyz="${xyz}" rpy="${rpy}" />
+            <mass value="${m}" />
+            <inertia ixx="${(2/5)*(m*r*r)}" ixy="0" ixz="0"
+                iyy="${(2/5)*(m*r*r)}" iyz="0"
+                izz="${(2/5)*(m*r*r)}" />
+        </inertial>
+    </xacro:macro>
 </robot>

File: src/my_robot_description/urdf/mobile_base.xacro (robot description, xacro)
@@ -20,4 +20,12 @@
             <material name="blue" />
         </visual>
+        <collision>
+            <geometry>
+                <box size="${base_length} ${base_width} ${base_height}" />
+            </geometry>
+            <origin xyz="0 0 ${base_height/ 2.0}" rpy="0 0 0" />
+        </collision>
+        <!-- mass in kg -->
+        <xacro:box_inertia m="5.0" l="${2*base_length}" w="${2*base_width}" h="${2*base_height}" xyz="0 0 ${base_height/ 2.0}" rpy="0 0 0" />
     </link>
     <xacro:macro name="wheel_link" params="prefix">
@@ -31,4 +39,11 @@
                 <material name="grey" />
             </visual>
+            <collision>
+                <geometry>
+                    <cylinder radius="${wheel_radius}" length="${wheel_length}" />
+                </geometry>
+                <origin xyz="0 0 0" rpy="${pi /2.0} 0 0" />
+            </collision>
+            <xacro:cylinder_inertia m="1.0" r="${2*wheel_radius}" h="${2*wheel_length}" xyz="0 0 0" rpy="${pi /2.0} 0 0" />
         </link>
     </xacro:macro>
@@ -43,4 +58,11 @@
             <material name="grey" />
         </visual>
+        <collision>
+            <geometry>
+                <sphere radius="${wheel_radius / 2.0}" />
+            </geometry>
+            <origin xyz="0 0 0" rpy="0 0 0" />
+        </collision>
+        <xacro:sphere_inertia m="0.5" r="${2 * wheel_radius / 2.0}" xyz="0 0 0" rpy="0 0 0" />
     </link>
     <joint name="base_joint" type="fixed">

File: src/my_robot_description/urdf/my_robot.urdf.xacro (robot description, xacro)
@@ -3,3 +3,5 @@
     <xacro:include filename="common_properties.xacro" />
     <xacro:include filename="mobile_base.xacro" />
+    <!-- Put the gazebo config after the robot definition -->
+    <xacro:include filename="mobile_base_gazebo.xacro" />
 </robot>

Commit message: 08 - Final Project

File: src/my_robot_description/urdf/common_properties.xacro (robot description, xacro)
@@ -6,4 +6,10 @@
     <material name="grey">
         <color rgba="0.5 0.5 0.5 1" />
+    </material>
+    <material name="orange">
+        <color rgba="1.0 0.5 0 1"/>
+    </material>
+    <material name="yellow">
+        <color rgba="1.0 1.0 0 1"/>
     </material>
     <xacro:macro name="box_inertia" params="m l w h xyz rpy">

File: src/my_robot_description/urdf/my_robot.urdf.xacro (robot description, xacro)
@@ -1,8 +1,16 @@
 <?xml version="1.0"?>
-<robot name="my_robot" xmlns:xacro="http:www.ros.org/wiki/xacro">
+<robot name="my_robot"
+    xmlns:xacro="http:www.ros.org/wiki/xacro">
     <xacro:include filename="common_properties.xacro" />
     <xacro:include filename="mobile_base.xacro" />
     <!-- Put the gazebo config after the robot definition -->
     <xacro:include filename="mobile_base_gazebo.xacro" />
+    <xacro:include filename="arm.xacro" />
+    <xacro:include filename="arm_gazebo.xacro" />
+    <joint name="mobile_base_arm_joint" type ="fixed">
+        <parent link="base_link"/>
+        <child link="arm_base_link" />
+        <origin xyz="${base_length / 4.0} 0 ${base_height}" rpy="0 0 0" />
+    </joint>
     <xacro:include filename="camera.xacro" />
 </robot>
